Commit message: Final Changes

File: kuka_lbr_iisy_support/urdf/lbr_iisy3_r760.urdf.xacro (robot description, xacro)
@@ -23,5 +23,4 @@
   <xacro:arg name="yaw" default="0"/>
   <xacro:kuka_lbr_iisy_ros2_control name="$(arg prefix)lbr_iisy3_r760" driver_version="$(arg driver_version)" client_ip="$(arg client_ip)" client_port="$(arg client_port)" mxa_client_port="$(arg mxa_client_port)" controller_ip="$(arg controller_ip)" prefix="$(arg prefix)" mode="$(arg mode)" use_gpio="$(arg use_gpio)" roundtrip_time="$(arg roundtrip_time)" verify_robot_model="$(arg verify_robot_model)" qos_config_file="$(arg qos_config_file)">
-    <ext_axes_ros2_control_joints/>
   </xacro:kuka_lbr_iisy_ros2_control>
   <!-- world link -->

File: kuka_lbr_iisy_support/urdf/lbr_iisy_ros2_control_macro.xacro (robot description, xacro)
@@ -1,5 +1,5 @@
 <?xml version="1.0" encoding="UTF-8"?>
 <robot xmlns:xacro="http://www.ros.org/wiki/xacro">
-  <xacro:macro name="kuka_lbr_iisy_ros2_control" params="name driver_version prefix client_ip client_port mxa_client_port controller_ip use_gpio mode qos_config_file roundtrip_time verify_robot_model **ext_axes_ros2_control_joints">
+  <xacro:macro name="kuka_lbr_iisy_ros2_control" params="name driver_version prefix client_ip client_port mxa_client_port controller_ip use_gpio mode qos_config_file roundtrip_time verify_robot_model">
     <!-- gazebo -->
     <xacro:if value="${mode == 'gazebo'}">
@@ -65,5 +65,4 @@
         </xacro:if>
       </hardware>
-      <xacro:insert_block name="ext_axes_ros2_control_joints"/>
       <!-- define joints and command/state interfaces for each joint -->
       <joint name="${prefix}joint_1">
@@ -79,7 +78,4 @@
         <xacro:if value="${driver_version == 'eac'}">
           <state_interface name="effort">
-            <param name="initial_value">0.0</param>
-          </state_interface>
-          <state_interface name="commanded_position">
             <param name="initial_value">0.0</param>
           </state_interface>
@@ -100,7 +96,4 @@
             <param name="initial_value">0.0</param>
           </state_interface>
-          <state_interface name="commanded_position">
-            <param name="initial_value">0.0</param>
-          </state_interface>
         </xacro:if>
       </joint>
@@ -117,7 +110,4 @@
         <xacro:if value="${driver_version == 'eac'}">
           <state_interface name="effort">
-            <param name="initial_value">0.0</param>
-          </state_interface>
-          <state_interface name="commanded_position">
             <param name="initial_value">0.0</param>
           </state_interface>
@@ -138,7 +128,4 @@
             <param name="initial_value">0.0</param>
           </state_interface>
-          <state_interface name="commanded_position">
-            <param name="initial_value">0.0</param>
-          </state_interface>
         </xacro:if>
       </joint>
@@ -155,7 +142,4 @@
         <xacro:if value="${driver_version == 'eac'}">
           <state_interface name="effort">
-            <param name="initial_value">0.0</param>
-          </state_interface>
-          <state_interface name="commanded_position">
             <param name="initial_value">0.0</param>
           </state_interface>
@@ -176,7 +160,4 @@
             <param name="initial_value">0.0</param>
           </state_interface>
-          <state_interface name="commanded_position">
-            <param name="initial_value">0.0</param>
-          </state_interface>
         </xacro:if>
       </joint>
